Commit message: Fixed frame id bugg and launch file

File: unicorn_description/urdf/stereo_camera.urdf.xacro (robot description, xacro)
@@ -14,5 +14,5 @@
         <!-- Origin of this mesh is the focal point of the LIDAR. -->
         <!-- <mesh filename="package://unicorn_description/stereo_camera_model/zed_model.dae" /> -->
-          <box size="${0.035} ${0.025} ${0.19}"/>
+          <box size="${0.005} ${0.025} ${0.19}"/>
         </geometry>
         <material name="red"/>

File: unicorn_description/urdf/unicorn_target.urdf.xacro (robot description, xacro)
@@ -29,5 +29,5 @@
   </macro>
   <link
-    name="chassis_link">
+    name="base_link">
     <inertial>
       <origin
@@ -68,52 +68,8 @@
     </collision>
   </link>
-  <link
-    name="base_link">
-    <inertial>
-      <origin
-        xyz="0.17 0 0"
-        rpy="0 0 0" />
-      <mass
-        value="0.01" />
-      <box_inertia  m="${5*0.01}" x="${base_x_size}" y="${base_y_size}" z="${base_z_size}"/>
-    </inertial>
-    <visual>
-      <origin
-        xyz="0 0 0"
-        rpy="0 0 0" />
-      <geometry>
-        <box size="0.01 0.01 0.01"/>
-      </geometry>
-      <material
-        name="">
-        <color
-          rgba="0.79216 0.81961 0.93333 1" />
-      </material>
-    </visual>
-    <collision>
-      <origin
-        xyz="0 0 0"
-        rpy="0 0 0" />
-      <geometry>
-        <!-- <mesh
-          filename="package://unicorn_description/meshes/base_link.STL" /> -->
-          <box size="0.01 0.01 0.01"/>
-      </geometry>
-      <!-- <surface>
-         <friction>
-           <ode><mu>0</mu><mu2>0</mu2></ode>
-         </friction>
-      </surface> -->
-    </collision>
-  </link>
   <gazebo reference="base_link_gazebo">
     <material>Gazebo/Green</material>
     <turnGravityOff>false</turnGravityOff>
   </gazebo>
-  <joint name="base_link_joint" type="fixed">
-    <parent link="chassis_link"/>
-    <child link="base_link_gazebo" />
-  <origin xyz="0 0.0 0" rpy="0 0 0" />
-  </joint>
   <!-- WHEELs -->
   <wheel fb="back" lr="right" parent="base_link" translateY="-0.24" translateX="0.0" translateZ="0.0" wheel_radius="0.1225" wheel_height="0.032" flip="1"/>

Commit message: Update unicorn_target.urdf.xacro to include zed

File: unicorn_description/urdf/stereo_camera.urdf.xacro (robot description, xacro)
@@ -1,2 +1,3 @@
+<?xml version="1.0"?>
 <robot xmlns:xacro="http://ros.org/wiki/xacro">
   <xacro:macro name="stereo_camera" params="frame topic:=pointcloud robot_namespace:=/" >

File: unicorn_description/urdf/unicorn_target.urdf.xacro (robot description, xacro)
@@ -14,4 +14,5 @@
   <xacro:include filename="$(find am_description)/urdf/sensorpos.urdf.xacro" />
   <xacro:include filename="$(find lms1xx)/urdf/sick_lms1xx.urdf.xacro" />
+  <xacro:include filename="$(find unicorn_description)/urdf/stereo_camera.urdf.xacro" />
   <!--<xacro:include filename="$(find husky_description)/urdf/accessories/sick_lms1xx_mount.urdf.xacro"/>-->
   <!--<xacro:include filename="$(find husky_description)/urdf/accessories/sensor_arch.urdf.xacro"/>-->
@@ -72,4 +73,58 @@
     <turnGravityOff>false</turnGravityOff>
   </gazebo>
+  <link name="zed_left_camera">
+        <visual>
+            <origin xyz="0 0 0" rpy="0 1.57 0"/>
+            <geometry>
+                <cylinder radius="0.007" length=".031"/>
+            </geometry>
+            <material name="dark_grey">
+                <color rgba="0.1 0.1 0.1 1"/>
+            </material>
+        </visual>
+    </link>
+    <link name="zed_center">
+        <visual>
+            <origin xyz="0 0 0" rpy="0 0 0"/>
+            <geometry>
+                <mesh filename="package://zed_wrapper/urdf/ZED.stl" />
+            </geometry>
+            <material name="light_grey">
+                <color rgba="0.8 0.8 0.8 0.8"/>
+            </material>
+        </visual>
+    </link>
+    <link name="zed_right_camera">
+        <visual>
+            <origin xyz="0 0 0" rpy="0 1.57 0"/>
+            <geometry>
+                <cylinder radius="0.007" length=".031"/>
+            </geometry>
+            <material name="dark_grey">
+                <color rgba="0.1 0.1 0.1 1"/>
+            </material>
+        </visual>
+    </link>
+    <link name="zed_depth_camera" />
+    <joint name="zed_left_camera_joint" type="fixed">
+        <parent link="zed_center"/>
+        <child link="zed_left_camera"/>
+        <origin xyz="0 0.06 0" rpy="0 0 0" />
+    </joint>
+    <joint name="zed_depth_camera_joint" type="fixed">
+        <parent link="zed_left_camera"/>
+        <child link="zed_depth_camera"/>
+        <origin xyz="0 0 0" rpy="-1.5707963267948966 0 -1.5707963267948966" />
+    </joint>
+    <joint name="zed_right_camera_joint" type="fixed">
+        <parent link="zed_center"/>
+        <child link="zed_right_camera"/>
+        <origin xyz="0 -0.06 0" rpy="0 0 0" />
+    </joint>
+    <joint name="zed_center_joint" type="fixed">
+      <parent link="base_link"/>
+      <child link="zed_center"/>
+      <origin xyz="0 0 0.3" rpy="${-M_PI/2} 0 0"/>
+    </joint>
   <!-- WHEELs -->
   <wheel fb="back" lr="right" parent="base_link" translateY="-0.24" translateX="0.0" translateZ="0.0" wheel_radius="0.1225" wheel_height="0.032" flip="1"/>

Commit message: Added ultrasonic sensors and depth camera to the gazeob simulation

File: unicorn_description/urdf/stereo_camera.urdf.xacro (robot description, xacro)
@@ -57,5 +57,5 @@
           <frameName>camera_left_depth_link</frameName>
           <robotNamespace>${robot_namespace}</robotNamespace>
-          <pointCloudCutoff>10.0</pointCloudCutoff>
+          <pointCloudCutoff>0.05</pointCloudCutoff>
           <distortionK1>0</distortionK1>
           <distortionK2>0</distortionK2>

File: unicorn_description/urdf/unicorn_2_back.urdf.xacro (robot description, xacro)
@@ -24,4 +24,9 @@
   <xacro:arg name="ultrasonic_rpy" default="0 0 ${M_PI}" />
   <xacro:include filename="$(find unicorn_description)/urdf/ultrasonic_sensor.urdf.xacro" />
+  <!-- Camera -->
+  <xacro:arg name="camera_enabled" default="true" />
+  <xacro:arg name="camera_xyz" default="0.3206 0.0 0.6" />
+  <xacro:arg name="camera_rpy" default="0.0 0.0 0.0" />
+  <xacro:include filename="$(find unicorn_description)/urdf/stereo_camera.urdf.xacro" />
   <!-- Wheel -->
   <xacro:include filename="$(find am_description)/urdf/wheel.urdf.xacro" />
@@ -176,5 +181,38 @@
     <child link="base_laser" />
   </joint>
-  <!-- Ultrasonic sensor -->
+  <!-- Camera -->
+  <xacro:if value="$(arg camera_enabled)">
+    <stereo_camera frame="camera_left_link" topic="pointcloud" robot_namespace="$(arg robot_namespace)"/>
+    <!-- generate an optical frame http://www.ros.org/reps/rep-0103.html#suffix-frames
+        so that ros and opencv can operate on the camera frame correctly -->
+    <joint name="camera_optical_joint" type="fixed">
+      <!-- these values have to be these values otherwise the gazebo camera image
+          won't be aligned properl  y with the frame it is supposedly originating from -->
+      <origin xyz="$(arg camera_xyz)" rpy="0 0 ${-pi}"/>
+      <parent link="base_link_gazebo"/>
+      <child link="camera_left_link"/>
+    </joint>
+    <joint name="camera_depth_joint" type="fixed">
+      <origin xyz="0 0 0" rpy="${-pi/2} 0 ${-pi/2}"/>
+      <parent link="camera_left_link"/>
+      <child link="camera_left_depth_link"/>
+    </joint>
+  </xacro:if>
+  <!-- GPS -->
+  <gazebo>
+    <plugin name="novatel_gps_sim" filename="libhector_gazebo_ros_gps.so">
+      <alwaysOn>1</alwaysOn>
+      <updateRate>10.0</updateRate>
+      <bodyName>chassis_link</bodyName>
+      <topicName>gps</topicName>
+      <velocityTopicName>gps_velocity</velocityTopicName>
+      <drift>5.0 5.0 5.0</drift>
+      <gaussianNoise>0.1 0.1 0.1</gaussianNoise>
+      <velocityDrift>0 0 0</velocityDrift>
+      <velocityGaussianNoise>0.1 0.1 0.1</velocityGaussianNoise>
+    </plugin>
+  </gazebo>
+  <!-- Ultrasonic sensors -->
+  <!--
   <ultrasonic_sensor frame="base_ultrasonic_fr" topic="fr" robot_namespace="$(arg robot_namespace)"/>
   <joint name="ultrasonic_mount_joint_fr" type="fixed">
@@ -237,4 +275,5 @@
     <child link="base_ultrasonic_bl" />
   </joint>
+  -->
   <!-- GAZEBO STUFF -->
   <gazebo>
