Commit message: Backwards driven model added [working sim] + amcl parameter tuning

File: unicorn_description/urdf/unicorn_2_back.urdf.xacro (robot description, xacro)
@@ -27,5 +27,5 @@
   <xacro:include filename="$(find am_description)/urdf/materials.urdf.xacro" />
   <link
-    name="base_link_gazebo">
+    name="chassis_link">
     <inertial>
       <origin
@@ -38,6 +38,6 @@
     <visual>
       <origin
-        xyz="0.17 0 0"
-        rpy="0 0 ${M_PI}" />
+        xyz="-0.17 0 0"
+        rpy="0 0 0" />
       <geometry>
         <mesh
@@ -52,6 +52,6 @@
     <collision>
       <origin
-        xyz="0.17 0 0.08"
-        rpy="0 0 ${M_PI}" />
+        xyz="-0.17 0 0.08"
+        rpy="0 0 0" />
       <geometry>
         <!-- <mesh
@@ -66,12 +66,56 @@
     </collision>
   </link>
+  <link
+    name="base_link_gazebo">
+    <inertial>
+      <origin
+        xyz="0.17 0 0"
+        rpy="0 0 0" />
+      <mass
+        value="0.01" />
+      <box_inertia  m="${5*0.01}" x="${base_x_size}" y="${base_y_size}" z="${base_z_size}"/>
+    </inertial>
+    <visual>
+      <origin
+        xyz="0 0 0"
+        rpy="0 0 0" />
+      <geometry>
+        <box size="0.01 0.01 0.01"/>
+      </geometry>
+      <material
+        name="">
+        <color
+          rgba="0.79216 0.81961 0.93333 1" />
+      </material>
+    </visual>
+    <collision>
+      <origin
+        xyz="0 0 0"
+        rpy="0 0 0" />
+      <geometry>
+        <!-- <mesh
+          filename="package://unicorn_description/meshes/base_link.STL" /> -->
+          <box size="0.01 0.01 0.01"/>
+      </geometry>
+      <!-- <surface>
+         <friction>
+           <ode><mu>0</mu><mu2>0</mu2></ode>
+         </friction>
+      </surface> -->
+    </collision>
+  </link>
   <gazebo reference="base_link_gazebo">
     <material>Gazebo/Green</material>
     <turnGravityOff>false</turnGravityOff>
   </gazebo>
+  <joint name="base_link_gazebo_joint" type="fixed">
+    <parent link="chassis_link"/>
+    <child link="base_link_gazebo" />
+  <origin xyz="0 0.0 0" rpy="0 0 ${M_PI}" />
+  </joint>
   <wheel fb="back" lr="right" parent="base_link_gazebo" translateY="-0.24" translateX="0.0" translateZ="-0.006" wheel_radius="0.1225" wheel_height="0.032" flip="1"/>
   <wheel fb="back" lr="left" parent="base_link_gazebo" translateY="0.24" translateX="0.0" translateZ="-0.006" wheel_radius="0.1225" wheel_height="0.032" flip="1"/>
-  <swivel_wheel fb="front" lr="right" parent="base_link_gazebo" translateY="-0.16" translateX="0.205" translateZ="0.03" wheel_radius="0.05" wheel_height="0.05" flip="0"/>
-  <swivel_wheel fb="front" lr="left" parent="base_link_gazebo" translateY="0.16" translateX="0.205" translateZ="0.03" wheel_radius="0.05" wheel_height="0.05" flip="0"/>
+  <swivel_wheel fb="front" lr="right" parent="base_link_gazebo" translateY="-0.16" translateX="0.355" translateZ="0.03" wheel_radius="0.05" wheel_height="0.05" flip="0"/>
+  <swivel_wheel fb="front" lr="left" parent="base_link_gazebo" translateY="0.16" translateX="0.355" translateZ="0.03" wheel_radius="0.05" wheel_height="0.05" flip="0"/>
   <!-- LOOP SENSORs -->
   <!-- <sensorpos name="loop_front_center" parent="base_link_gazebo" translateX="0.38" translateY="0.0" translateZ="-0.04"/>
@@ -94,6 +138,6 @@
         <material name="Purple" />
     </visual>
-  </link> -->
-  <!-- <gazebo reference="cutting_disc_center">
+  </link>
+  <gazebo reference="cutting_disc_center">
     <turnGravityOff>false</turnGravityOff>
   </gazebo>
@@ -138,8 +182,8 @@
       <wheelDiameter>0.245</wheelDiameter>
       <wheelTorque>100</wheelTorque>
-      <commandTopic>/unicorn/cmd_vel</commandTopic>
+      <commandTopic>cmd_vel</commandTopic>
       <odometryTopic>odom</odometryTopic>
       <odometryFrame>odom_gazebo</odometryFrame>
-      <robotBaseFrame>base_footprint</robotBaseFrame>
+      <robotBaseFrame>chassis_link</robotBaseFrame>
       <publishWheelTF>false</publishWheelTF>
       <publishWheelJointState>false</publishWheelJointState>
@@ -148,5 +192,5 @@
     <plugin name="imu_plugin" filename="libhector_gazebo_ros_imu.so">
     <alwaysOn>false</alwaysOn>
-    <bodyName>base_link_gazebo</bodyName>
+    <bodyName>chassis_link</bodyName>
     <topicName>imu</topicName>
     <serviceName>imu_service</serviceName>

File: unicorn_description/urdf/unicorn_2_safe.urdf.xacro (robot description, xacro)
@@ -18,5 +18,5 @@
   <!-- LMS111 -->
   <xacro:arg name="laser_xyz" default="0.0 0.0 0.260" />
-  <xacro:arg name="laser_rpy" default="0.0 0.0 ${M_PI}" />
+  <xacro:arg name="laser_rpy" default="0.0 0.0 0.0" />
   <xacro:include filename="$(find lms1xx)/urdf/sick_lms1xx.urdf.xacro" />
   <!-- Wheel -->
@@ -38,6 +38,6 @@
     <visual>
       <origin
-        xyz="0.17 0 0"
-        rpy="0 0 ${M_PI}" />
+        xyz="-0.205 0 0"
+        rpy="0 0 0" />
       <geometry>
         <mesh
@@ -52,6 +52,6 @@
     <collision>
       <origin
-        xyz="0.17 0 0.08"
-        rpy="0 0 ${M_PI}" />
+        xyz="-0.205 0 0.08"
+        rpy="0 0 0" />
       <geometry>
         <!-- <mesh
@@ -59,9 +59,9 @@
           <box size="0.65 0.5 0.2"/>
       </geometry>
-      <!-- <surface>
-         <friction>
-           <ode><mu>0</mu><mu2>0</mu2></ode>
-         </friction>
-      </surface> -->
+	    <!-- <surface>
+	       <friction>
+	         <ode><mu>0</mu><mu2>0</mu2></ode>
+	       </friction>
+	    </surface> -->
     </collision>
   </link>
@@ -72,6 +72,6 @@
   <wheel fb="back" lr="right" parent="base_link_gazebo" translateY="-0.24" translateX="0.0" translateZ="-0.006" wheel_radius="0.1225" wheel_height="0.032" flip="1"/>
   <wheel fb="back" lr="left" parent="base_link_gazebo" translateY="0.24" translateX="0.0" translateZ="-0.006" wheel_radius="0.1225" wheel_height="0.032" flip="1"/>
-  <swivel_wheel fb="front" lr="right" parent="base_link_gazebo" translateY="-0.16" translateX="0.205" translateZ="0.03" wheel_radius="0.05" wheel_height="0.05" flip="0"/>
-  <swivel_wheel fb="front" lr="left" parent="base_link_gazebo" translateY="0.16" translateX="0.205" translateZ="0.03" wheel_radius="0.05" wheel_height="0.05" flip="0"/>
+  <swivel_wheel fb="front" lr="right" parent="base_link_gazebo" translateY="-0.16" translateX="-0.355" translateZ="0.03" wheel_radius="0.05" wheel_height="0.05" flip="0"/>
+  <swivel_wheel fb="front" lr="left" parent="base_link_gazebo" translateY="0.16" translateX="-0.355" translateZ="0.03" wheel_radius="0.05" wheel_height="0.05" flip="0"/>
   <!-- LOOP SENSORs -->
   <!-- <sensorpos name="loop_front_center" parent="base_link_gazebo" translateX="0.38" translateY="0.0" translateZ="-0.04"/>
@@ -94,6 +94,6 @@
         <material name="Purple" />
     </visual>
-  </link> -->
-  <!-- <gazebo reference="cutting_disc_center">
+  </link>
+  <gazebo reference="cutting_disc_center">
     <turnGravityOff>false</turnGravityOff>
   </gazebo>
@@ -138,5 +138,5 @@
       <wheelDiameter>0.245</wheelDiameter>
       <wheelTorque>100</wheelTorque>
-      <commandTopic>/unicorn/cmd_vel</commandTopic>
+      <commandTopic>cmd_vel</commandTopic>
       <odometryTopic>odom</odometryTopic>
       <odometryFrame>odom_gazebo</odometryFrame>

File: unicorn_description/urdf/unicorn_target_2.urdf.xacro (robot description, xacro)
@@ -27,5 +27,5 @@
   <xacro:include filename="$(find am_description)/urdf/materials.urdf.xacro" />
   <link
-    name="base_link_gazebo">
+    name="chassis_link">
     <inertial>
       <origin
@@ -38,6 +38,6 @@
     <visual>
       <origin
-        xyz="0.17 0 0"
-        rpy="0 0 ${M_PI}" />
+        xyz="-0.17 0 0"
+        rpy="0 0 0" />
       <geometry>
         <mesh
@@ -52,6 +52,6 @@
     <collision>
       <origin
-        xyz="0.17 0 0.08"
-        rpy="0 0 ${M_PI}" />
+        xyz="-0.17 0 0.08"
+        rpy="0 0 0" />
       <geometry>
         <!-- <mesh
@@ -66,23 +66,67 @@
     </collision>
   </link>
-  <gazebo reference="base_link_gazebo">
+  <link
+    name="base_link">
+    <inertial>
+      <origin
+        xyz="0.17 0 0"
+        rpy="0 0 0" />
+      <mass
+        value="0.01" />
+      <box_inertia  m="${5*0.01}" x="${base_x_size}" y="${base_y_size}" z="${base_z_size}"/>
+    </inertial>
+    <visual>
+      <origin
+        xyz="0 0 0"
+        rpy="0 0 0" />
+      <geometry>
+        <box size="0.01 0.01 0.01"/>
+      </geometry>
+      <material
+        name="">
+        <color
+          rgba="0.79216 0.81961 0.93333 1" />
+      </material>
+    </visual>
+    <collision>
+      <origin
+        xyz="0 0 0"
+        rpy="0 0 0" />
+      <geometry>
+        <!-- <mesh
+          filename="package://unicorn_description/meshes/base_link.STL" /> -->
+          <box size="0.01 0.01 0.01"/>
+      </geometry>
+      <!-- <surface>
+         <friction>
+           <ode><mu>0</mu><mu2>0</mu2></ode>
+         </friction>
+      </surface> -->
+    </collision>
+  </link>
+  <gazebo reference="base_link">
     <material>Gazebo/Green</material>
     <turnGravityOff>false</turnGravityOff>
   </gazebo>
-  <wheel fb="back" lr="right" parent="base_link_gazebo" translateY="-0.24" translateX="0.0" translateZ="-0.006" wheel_radius="0.1225" wheel_height="0.032" flip="1"/>
-  <wheel fb="back" lr="left" parent="base_link_gazebo" translateY="0.24" translateX="0.0" translateZ="-0.006" wheel_radius="0.1225" wheel_height="0.032" flip="1"/>
-  <swivel_wheel fb="front" lr="right" parent="base_link_gazebo" translateY="-0.16" translateX="0.205" translateZ="0.03" wheel_radius="0.05" wheel_height="0.05" flip="0"/>
-  <swivel_wheel fb="front" lr="left" parent="base_link_gazebo" translateY="0.16" translateX="0.205" translateZ="0.03" wheel_radius="0.05" wheel_height="0.05" flip="0"/>
+  <joint name="base_link_joint" type="fixed">
+    <parent link="chassis_link"/>
+    <child link="base_link" />
+  <origin xyz="0 0.0 0" rpy="0 0 ${M_PI}" />
+  </joint>
+  <wheel fb="back" lr="right" parent="base_link" translateY="-0.24" translateX="0.0" translateZ="-0.006" wheel_radius="0.1225" wheel_height="0.032" flip="1"/>
+  <wheel fb="back" lr="left" parent="base_link" translateY="0.24" translateX="0.0" translateZ="-0.006" wheel_radius="0.1225" wheel_height="0.032" flip="1"/>
+  <swivel_wheel fb="front" lr="right" parent="base_link" translateY="-0.16" translateX="0.355" translateZ="0.03" wheel_radius="0.05" wheel_height="0.05" flip="0"/>
+  <swivel_wheel fb="front" lr="left" parent="base_link" translateY="0.16" translateX="0.355" translateZ="0.03" wheel_radius="0.05" wheel_height="0.05" flip="0"/>
   <!-- LOOP SENSORs -->
-  <!-- <sensorpos name="loop_front_center" parent="base_link_gazebo" translateX="0.38" translateY="0.0" translateZ="-0.04"/>
-  <sensorpos name="loop_front_right" parent="base_link_gazebo" translateX="0.38" translateY="-0.07" translateZ="-0.04"/>
-  <sensorpos name="loop_rear_left" parent="base_link_gazebo" translateX="-0.07" translateY="0.14" translateZ="-0.04"/>
-  <sensorpos name="loop_rear_right" parent="base_link_gazebo" translateX="-0.07" translateY="-0.14" translateZ="-0.04"/> -->
+  <!-- <sensorpos name="loop_front_center" parent="base_link" translateX="0.38" translateY="0.0" translateZ="-0.04"/>
+  <sensorpos name="loop_front_right" parent="base_link" translateX="0.38" translateY="-0.07" translateZ="-0.04"/>
+  <sensorpos name="loop_rear_left" parent="base_link" translateX="-0.07" translateY="0.14" translateZ="-0.04"/>
+  <sensorpos name="loop_rear_right" parent="base_link" translateX="-0.07" translateY="-0.14" translateZ="-0.04"/> -->
   <!-- CONFINEMENT SENSORs -->
-  <!-- <sensorpos name="col_front_chassis" parent="base_link_gazebo" translateX="0.55" translateY="0.0" translateZ="0.00"/>
-  <sensorpos name="col_front_left" parent="base_link_gazebo" translateX="0.43" translateY="0.24" translateZ="0.00"/>
-  <sensorpos name="col_front_right" parent="base_link_gazebo" translateX="0.43" translateY="-0.24" translateZ="0.00"/>
-  <sensorpos name="col_rear_left" parent="base_link_gazebo" translateX="-0.10" translateY="0.24" translateZ="0.0"/>
-  <sensorpos name="col_rear_right" parent="base_link_gazebo" translateX="-0.10" translateY="-0.24" translateZ="0.0"/> -->
+  <!-- <sensorpos name="col_front_chassis" parent="base_link" translateX="0.55" translateY="0.0" translateZ="0.00"/>
+  <sensorpos name="col_front_left" parent="base_link" translateX="0.43" translateY="0.24" translateZ="0.00"/>
+  <sensorpos name="col_front_right" parent="base_link" translateX="0.43" translateY="-0.24" translateZ="0.00"/>
+  <sensorpos name="col_rear_left" parent="base_link" translateX="-0.10" translateY="0.24" translateZ="0.0"/>
+  <sensorpos name="col_rear_right" parent="base_link" translateX="-0.10" translateY="-0.24" translateZ="0.0"/> -->
   <!-- CUTTING DISC -->
   <!-- <link name="cutting_disc_center">
@@ -94,10 +138,10 @@
         <material name="Purple" />
     </visual>
-  </link> -->
-  <!-- <gazebo reference="cutting_disc_center">
+  </link>
+  <gazebo reference="cutting_disc_center">
     <turnGravityOff>false</turnGravityOff>
   </gazebo>
   <joint name="cutting_disc_center_joint" type="fixed">
-    <parent link="base_link_gazebo"/>
+    <parent link="base_link"/>
     <child link="cutting_disc_center" />
   <origin xyz="0.25 0.0 -0.07" rpy="0 0 0" />
@@ -117,5 +161,5 @@
   </gazebo>
   <joint name="antenna_center_joint" type="fixed">
-    <parent link="base_link_gazebo"/>
+    <parent link="base_link"/>
     <child link="antenna_center" />
   <origin xyz="0.27 0.0 0.0" rpy="0 0 0" />
@@ -125,5 +169,5 @@
     <joint name="laser_mount_joint" type="fixed">
       <origin xyz="$(arg laser_xyz)" rpy="$(arg laser_rpy)" />
-      <parent link="base_link_gazebo" />
+      <parent link="base_link" />
       <child link="base_laser" />
     </joint>
@@ -138,8 +182,8 @@
       <wheelDiameter>0.245</wheelDiameter>
       <wheelTorque>100</wheelTorque>
-      <commandTopic>/unicorn/cmd_vel</commandTopic>
+      <commandTopic>cmd_vel</commandTopic>
       <odometryTopic>odom</odometryTopic>
       <odometryFrame>odom_gazebo</odometryFrame>
-      <robotBaseFrame>base_footprint</robotBaseFrame>
+      <robotBaseFrame>chassis_link_gazebo</robotBaseFrame>
       <publishWheelTF>false</publishWheelTF>
       <publishWheelJointState>false</publishWheelJointState>
@@ -148,5 +192,5 @@
     <plugin name="imu_plugin" filename="libhector_gazebo_ros_imu.so">
     <alwaysOn>false</alwaysOn>
-    <bodyName>base_link_gazebo</bodyName>
+    <bodyName>chassis_link_gazebo</bodyName>
     <topicName>imu</topicName>
     <serviceName>imu_service</serviceName>

Commit message: Add ultrasonic sensor urdf

File: unicorn_description/urdf/unicorn_2_back.urdf.xacro (robot description, xacro)
@@ -20,4 +20,8 @@
   <xacro:arg name="laser_rpy" default="0.0 0.0 ${M_PI}" />
   <xacro:include filename="$(find lms1xx)/urdf/sick_lms1xx.urdf.xacro" />
+  <!-- Ultrasonic sensor -->
+  <xacro:arg name="ultrasonic_xyz" default="-0.3 0 0.2" />
+  <xacro:arg name="ultrasonic_rpy" default="0 0 ${M_PI}" />
+  <xacro:include filename="$(find unicorn_description)/urdf/ultrasonic_sensor.urdf.xacro" />
   <!-- Wheel -->
   <xacro:include filename="$(find am_description)/urdf/wheel.urdf.xacro" />
@@ -166,10 +170,71 @@
   </joint> -->
   <!--<sick_lms1xx_mount prefix="base"/>-->
-    <sick_lms1xx frame="base_laser" topic="scan" robot_namespace="$(arg robot_namespace)"/>
-    <joint name="laser_mount_joint" type="fixed">
-      <origin xyz="$(arg laser_xyz)" rpy="$(arg laser_rpy)" />
-      <parent link="base_link_gazebo" />
-      <child link="base_laser" />
-    </joint>
+  <sick_lms1xx frame="base_laser" topic="scan" robot_namespace="$(arg robot_namespace)"/>
+  <joint name="laser_mount_joint" type="fixed">
+    <origin xyz="$(arg laser_xyz)" rpy="$(arg laser_rpy)" />
+    <parent link="base_link_gazebo" />
+    <child link="base_laser" />
+  </joint>
+  <!-- Ultrasonic sensor -->
+  <ultrasonic_sensor frame="base_ultrasonic_fr" topic="fr" robot_namespace="$(arg robot_namespace)"/>
+  <joint name="ultrasonic_mount_joint_fr" type="fixed">
+    <origin xyz="-0.2 0.2 0.0" rpy="0 0 ${M_PI + M_PI/4}"/>
+    <parent link="base_link_gazebo"/>
+    <child link="base_ultrasonic_fr" />
+  </joint>
+  <ultrasonic_sensor frame="base_ultrasonic_fm" topic="fm" robot_namespace="$(arg robot_namespace)"/>
+  <joint name="ultrasonic_mount_joint_fm" type="fixed">
+    <origin xyz="-0.2 0.0 0.0" rpy="0 0 ${M_PI}"/>
+    <parent link="base_link_gazebo"/>
+    <child link="base_ultrasonic_fm" />
+  </joint>
+  <ultrasonic_sensor frame="base_ultrasonic_fl" topic="fl" robot_namespace="$(arg robot_namespace)"/>
+  <joint name="ultrasonic_mount_joint_fl" type="fixed">
+    <origin xyz="-0.2 -0.2 0.0" rpy="0 0 ${M_PI - M_PI/4}"/>
+    <parent link="base_link_gazebo"/>
+    <child link="base_ultrasonic_fl" />
+  </joint>
+  <ultrasonic_sensor frame="base_ultrasonic_r" topic="r" robot_namespace="$(arg robot_namespace)"/>
+  <joint name="ultrasonic_mount_joint_r" type="fixed">
+    <origin xyz="0.4 0.25 0.0" rpy="0 -${M_PI/64} ${3*M_PI/4}"/>
+    <parent link="base_link_gazebo"/>
+    <child link="base_ultrasonic_r" />
+  </joint>
+  <ultrasonic_sensor frame="base_ultrasonic_l" topic="l" robot_namespace="$(arg robot_namespace)"/>
+  <joint name="ultrasonic_mount_joint_l" type="fixed">
+    <origin xyz="0.4 -0.25 0.0" rpy="0 -${M_PI/64} -${3*M_PI/4}"/>
+    <parent link="base_link_gazebo"/>
+    <child link="base_ultrasonic_l" />
+  </joint>
+  <ultrasonic_sensor frame="base_ultrasonic_rm" topic="rm" robot_namespace="$(arg robot_namespace)"/>
+  <joint name="ultrasonic_mount_joint_rm" type="fixed">
+    <origin xyz="0.15 0.25 0.0" rpy="0 -${M_PI/64} ${M_PI/4}"/>
+    <parent link="base_link_gazebo"/>
+    <child link="base_ultrasonic_rm" />
+  </joint>
+  <ultrasonic_sensor frame="base_ultrasonic_lm" topic="lm" robot_namespace="$(arg robot_namespace)"/>
+  <joint name="ultrasonic_mount_joint_lm" type="fixed">
+    <origin xyz="0.15 -0.25 0.0" rpy="0 -${M_PI/64} -${M_PI/4}"/>
+    <parent link="base_link_gazebo"/>
+    <child link="base_ultrasonic_lm"/>
+  </joint>
+  <ultrasonic_sensor frame="base_ultrasonic_br" topic="br" robot_namespace="$(arg robot_namespace)"/>
+  <joint name="ultrasonic_mount_joint_br" type="fixed">
+    <origin xyz="0.5 0.2 0.0" rpy="0 -${M_PI/64} -${M_PI/4}"/>
+    <parent link="base_link_gazebo"/>
+    <child link="base_ultrasonic_br" />
+  </joint>
+  <ultrasonic_sensor frame="base_ultrasonic_bm" topic="bm" robot_namespace="$(arg robot_namespace)"/>
+  <joint name="ultrasonic_mount_joint_bm" type="fixed">
+    <origin xyz="0.5 0.0 0.0" rpy="0 -${M_PI/64} 0"/>
+    <parent link="base_link_gazebo"/>
+    <child link="base_ultrasonic_bm" />
+  </joint>
+  <ultrasonic_sensor frame="base_ultrasonic_bl" topic="bl" robot_namespace="$(arg robot_namespace)"/>
+  <joint name="ultrasonic_mount_joint_bl" type="fixed">
+    <origin xyz="0.5 -0.2 0.0" rpy="0 -${M_PI/64} ${M_PI/4}"/>
+    <parent link="base_link_gazebo"/>
+    <child link="base_ultrasonic_bl" />
+  </joint>
   <!-- GAZEBO STUFF -->
   <gazebo>

Commit message: Update range_sensor_driver and unicorn_statemachine [tested and working]

File: unicorn_description/urdf/unicorn_2_back.urdf.xacro (robot description, xacro)
@@ -25,5 +25,5 @@
   <xacro:include filename="$(find unicorn_description)/urdf/ultrasonic_sensor.urdf.xacro" />
   <!-- Camera -->
-  <xacro:arg name="camera_enabled" default="true" />
+  <xacro:arg name="camera_enabled" default="false" />
   <xacro:arg name="camera_xyz" default="0.3206 0.0 0.6" />
   <xacro:arg name="camera_rpy" default="0.0 0.0 0.0" />
@@ -214,5 +214,4 @@
   </gazebo>
   <!-- Ultrasonic sensors -->
-  <!--
   <ultrasonic_sensor frame="base_ultrasonic_fr" topic="fr" robot_namespace="$(arg robot_namespace)"/>
   <joint name="ultrasonic_mount_joint_fr" type="fixed">
@@ -275,5 +274,4 @@
     <child link="base_ultrasonic_bl" />
   </joint>
-  -->
   <!-- GAZEBO STUFF -->
   <gazebo>

File: unicorn_description/urdf/unicorn_target_2.urdf.xacro (robot description, xacro)
@@ -166,5 +166,5 @@
       <parent link="chassis_link"/>
       <child link="zed_center"/>
-      <origin xyz="-0.2 0.0 0.0" rpy="0 0 ${-M_PI}"/>
+      <origin xyz="-0.2 0.0 0.3" rpy="0 0 ${-M_PI}"/>
     </joint>
   <!-- Orbbec camera -->
