Commit message: Add backwards driving support for automower [working]

File: unicorn_description/urdf/unicorn_target_2.urdf.xacro (robot description, xacro)
@@ -27,8 +27,8 @@
   <xacro:include filename="$(find am_description)/urdf/materials.urdf.xacro" />
   <link
-    name="chassis_link">
+    name="base_link">
     <inertial>
       <origin
-        xyz="0.17 0 -0.10"
+        xyz="0 0 0"
         rpy="0 0 0" />
       <mass
@@ -67,5 +67,5 @@
   </link>
   <link
-    name="base_link">
+    name="chassis_link">
     <inertial>
       <origin
@@ -105,17 +105,71 @@
     </collision>
   </link>
-  <gazebo reference="base_link">
+  <gazebo reference="base_link_gazebo">
     <material>Gazebo/Green</material>
     <turnGravityOff>false</turnGravityOff>
   </gazebo>
-  <joint name="base_link_joint" type="fixed">
-    <parent link="chassis_link"/>
-    <child link="base_link" />
+  <joint name="base_chassis_joint" type="fixed">
+    <parent link="base_link"/>
+    <child link="chassis_link" />
   <origin xyz="0 0.0 0" rpy="0 0 ${M_PI}" />
   </joint>
-  <wheel fb="back" lr="right" parent="base_link" translateY="-0.24" translateX="0.0" translateZ="-0.006" wheel_radius="0.1225" wheel_height="0.032" flip="1"/>
-  <wheel fb="back" lr="left" parent="base_link" translateY="0.24" translateX="0.0" translateZ="-0.006" wheel_radius="0.1225" wheel_height="0.032" flip="1"/>
-  <swivel_wheel fb="front" lr="right" parent="base_link" translateY="-0.16" translateX="0.355" translateZ="0.03" wheel_radius="0.05" wheel_height="0.05" flip="0"/>
-  <swivel_wheel fb="front" lr="left" parent="base_link" translateY="0.16" translateX="0.355" translateZ="0.03" wheel_radius="0.05" wheel_height="0.05" flip="0"/>
+  <link name="zed_left_camera">
+        <visual>
+            <origin xyz="0 0 0" rpy="0 1.57 0"/>
+            <geometry>
+                <cylinder radius="0.007" length=".031"/>
+            </geometry>
+            <material name="dark_grey">
+                <color rgba="0.1 0.1 0.1 1"/>
+            </material>
+        </visual>
+    </link>
+    <link name="zed_center">
+        <visual>
+            <origin xyz="0 0 0" rpy="0 0 0"/>
+            <geometry>
+                <mesh filename="package://zed_wrapper/urdf/ZED.stl" />
+            </geometry>
+            <material name="light_grey">
+                <color rgba="0.8 0.8 0.8 0.8"/>
+            </material>
+        </visual>
+    </link>
+    <!-- <link name="zed_right_camera">
+        <visual>
+            <origin xyz="0 0 0" rpy="0 1.57 0"/>
+            <geometry>
+                <cylinder radius="0.007" length=".031"/>
+            </geometry>
+            <material name="dark_grey">
+                <color rgba="0.1 0.1 0.1 1"/>
+            </material>
+        </visual>
+    </link> -->
+    <link name="zed_depth_camera" />
+    <joint name="zed_left_camera_joint" type="fixed">
+        <parent link="zed_center"/>
+        <child link="zed_left_camera"/>
+        <origin xyz="0 0.06 0" rpy="0 0 0" />
+    </joint>
+    <joint name="zed_depth_camera_joint" type="fixed">
+        <parent link="zed_left_camera"/>
+        <child link="zed_depth_camera"/>
+        <origin xyz="0 0 0" rpy="-1.5707963267948966 0 -1.5707963267948966" />
+    </joint>
+   <!--  <joint name="zed_right_camera_joint" type="fixed">
+        <parent link="zed_center"/>
+        <child link="zed_right_camera"/>
+        <origin xyz="0 -0.06 0" rpy="0 0 0" />
+    </joint> -->
+    <joint name="chassis_zed_joint" type="fixed">
+      <parent link="chassis_link"/>
+      <child link="zed_center"/>
+      <origin xyz="0 0 0.3" rpy="0 0 0"/>
+    </joint>
+  <wheel fb="back" lr="right" parent="chassis_link" translateY="-0.24" translateX="0.0" translateZ="-0.006" wheel_radius="0.1225" wheel_height="0.032" flip="1"/>
+  <wheel fb="back" lr="left" parent="chassis_link" translateY="0.24" translateX="0.0" translateZ="-0.006" wheel_radius="0.1225" wheel_height="0.032" flip="1"/>
+  <swivel_wheel fb="front" lr="right" parent="chassis_link" translateY="-0.16" translateX="0.355" translateZ="0.03" wheel_radius="0.05" wheel_height="0.05" flip="0"/>
+  <swivel_wheel fb="front" lr="left" parent="chassis_link" translateY="0.16" translateX="0.355" translateZ="0.03" wheel_radius="0.05" wheel_height="0.05" flip="0"/>
   <!-- LOOP SENSORs -->
   <!-- <sensorpos name="loop_front_center" parent="base_link" translateX="0.38" translateY="0.0" translateZ="-0.04"/>
@@ -169,5 +223,5 @@
     <joint name="laser_mount_joint" type="fixed">
       <origin xyz="$(arg laser_xyz)" rpy="$(arg laser_rpy)" />
-      <parent link="base_link" />
+      <parent link="chassis_link" />
       <child link="base_laser" />
     </joint>

Commit message: Tune costmap params, amcl params, and use teb local planner [tested and working]

File: unicorn_description/urdf/unicorn_target_2.urdf.xacro (robot description, xacro)
@@ -17,5 +17,5 @@
   </macro>
   <!-- LMS111 -->
-  <xacro:arg name="laser_xyz" default="0.0 0.0 0.260" />
+  <xacro:arg name="laser_xyz" default="0.0 0.0 0.5" />
   <xacro:arg name="laser_rpy" default="0.0 0.0 ${M_PI}" />
   <xacro:include filename="$(find lms1xx)/urdf/sick_lms1xx.urdf.xacro" />
@@ -30,5 +30,5 @@
     <inertial>
       <origin
-        xyz="0 0 0"
+        xyz="0.17 0 0"
         rpy="0 0 0" />
       <mass
@@ -70,5 +70,5 @@
     <inertial>
       <origin
-        xyz="0.17 0 0"
+        xyz="0 0 0"
         rpy="0 0 0" />
       <mass
@@ -166,10 +166,10 @@
       <parent link="chassis_link"/>
       <child link="zed_center"/>
-      <origin xyz="0 0 0.3" rpy="0 0 0"/>
-    </joint>
-  <wheel fb="back" lr="right" parent="chassis_link" translateY="-0.24" translateX="0.0" translateZ="-0.006" wheel_radius="0.1225" wheel_height="0.032" flip="1"/>
-  <wheel fb="back" lr="left" parent="chassis_link" translateY="0.24" translateX="0.0" translateZ="-0.006" wheel_radius="0.1225" wheel_height="0.032" flip="1"/>
-  <swivel_wheel fb="front" lr="right" parent="chassis_link" translateY="-0.16" translateX="0.355" translateZ="0.03" wheel_radius="0.05" wheel_height="0.05" flip="0"/>
-  <swivel_wheel fb="front" lr="left" parent="chassis_link" translateY="0.16" translateX="0.355" translateZ="0.03" wheel_radius="0.05" wheel_height="0.05" flip="0"/>
+      <origin xyz="0.2 0 0.3" rpy="0 0 ${M_PI}"/>
+    </joint>
+  <wheel fb="back" lr="left" parent="chassis_link" translateY="-0.24" translateX="0.0" translateZ="-0.006" wheel_radius="0.1225" wheel_height="0.032" flip="1"/>
+  <wheel fb="back" lr="right" parent="chassis_link" translateY="0.24" translateX="0.0" translateZ="-0.006" wheel_radius="0.1225" wheel_height="0.032" flip="1"/>
+  <swivel_wheel fb="front" lr="left" parent="chassis_link" translateY="-0.16" translateX="0.355" translateZ="0.03" wheel_radius="0.05" wheel_height="0.05" flip="0"/>
+  <swivel_wheel fb="front" lr="right" parent="chassis_link" translateY="0.16" translateX="0.355" translateZ="0.03" wheel_radius="0.05" wheel_height="0.05" flip="0"/>
   <!-- LOOP SENSORs -->
   <!-- <sensorpos name="loop_front_center" parent="base_link" translateX="0.38" translateY="0.0" translateZ="-0.04"/>

Commit message: Added the frames for the orbbec

File: unicorn_description/urdf/unicorn_target_2.urdf.xacro (robot description, xacro)
@@ -168,4 +168,55 @@
       <origin xyz="0.2 0 0.3" rpy="0 0 ${M_PI}"/>
     </joint>
+  <!-- Orbbec camera -->
+  <link name="camera_rgb_frame">
+      <visual>
+          <origin xyz="0 0 0" rpy="0 1.57 0"/>
+          <geometry>
+              <box size="0.01 0.01 0.01"/>
+          </geometry>
+          <material name="dark_grey">
+              <color rgba="0.1 0.1 0.1 1"/>
+          </material>
+      </visual>
+  </link>
+  <link name="camera_link">
+      <visual>
+          <origin xyz="0 0 0" rpy="0 0 0"/>
+          <geometry>
+              <box size="0.01 0.01 0.01"/>
+          </geometry>
+          <material name="light_grey">
+              <color rgba="0.8 0.8 0.8 0.8"/>
+          </material>
+      </visual>
+  </link>
+  <link name="camera_depth_frame" />
+  <link name="camera_depth_optical_frame" />
+  <link name="camera_rgb_optical_frame" />
+  <joint name="chassis_orbbec_joint" type="fixed">
+    <parent link="chassis_link"/>
+    <child link="camera_link"/>
+    <origin xyz="0.2 0 0.3" rpy="0 0 ${M_PI}"/>
+  </joint>
+  <joint name="orbbec_rgb_camera_joint" type="fixed">
+    <parent link="camera_link"/>
+    <child link="camera_rgb_frame"/>
+    <origin xyz="0 0.06 0" rpy="0 0 0" />
+  </joint>
+  <joint name="orbbec_depth_camera_joint" type="fixed">
+    <parent link="camera_link"/>
+    <child link="camera_depth_frame"/>
+    <origin xyz="0 0 0" rpy="-1.5707963267948966 0 -1.5707963267948966" />
+  </joint>
+  <joint name="orbbec_depth_optical_joint" type="fixed">
+    <parent link="camera_depth_frame"/>
+    <child link="camera_depth_optical_frame"/>
+    <origin xyz="0 0 0" rpy="0 0 0" />
+  </joint>
+  <joint name="orbbec_rgb_optical_joint" type="fixed">
+    <parent link="camera_rgb_frame"/>
+    <child link="camera_rgb_optical_frame"/>
+    <origin xyz="0 0 0" rpy="0 0 0" />
+  </joint>
   <wheel fb="back" lr="left" parent="chassis_link" translateY="-0.24" translateX="0.0" translateZ="-0.006" wheel_radius="0.1225" wheel_height="0.032" flip="1"/>
   <wheel fb="back" lr="right" parent="chassis_link" translateY="0.24" translateX="0.0" translateZ="-0.006" wheel_radius="0.1225" wheel_height="0.032" flip="1"/>

Commit message: Fix bugg where laser and pointcloud were not aligned

File: unicorn_description/urdf/unicorn_target_2.urdf.xacro (robot description, xacro)
@@ -166,5 +166,5 @@
       <parent link="chassis_link"/>
       <child link="zed_center"/>
-      <origin xyz="0.2 0 0.3" rpy="0 0 ${M_PI}"/>
+      <origin xyz="-0.2 0.0 0.0" rpy="0 0 ${-M_PI}"/>
     </joint>
   <!-- Orbbec camera -->

Commit message: Update range sensor driver to get topic parameter from sonar_layer + update how to input parameters to laser_filter node

File: unicorn_description/urdf/unicorn_target_2.urdf.xacro (robot description, xacro)
@@ -20,4 +20,8 @@
   <xacro:arg name="laser_rpy" default="0.0 0.0 ${M_PI}" />
   <xacro:include filename="$(find lms1xx)/urdf/sick_lms1xx.urdf.xacro" />
+  <!-- Ultrasonic sensor -->
+  <xacro:arg name="ultrasonic_xyz" default="-0.3 0 0.2" />
+  <xacro:arg name="ultrasonic_rpy" default="0 0 0" />
+  <xacro:include filename="$(find unicorn_description)/urdf/ultrasonic_sensor.urdf.xacro" />
   <!-- Wheel -->
   <xacro:include filename="$(find am_description)/urdf/wheel.urdf.xacro" />
@@ -270,5 +274,10 @@
   <origin xyz="0.27 0.0 0.0" rpy="0 0 0" />
   </joint> -->
-  <!--<sick_lms1xx_mount prefix="base"/>-->
+  <ultrasonic_sensor frame="base_ultrasonic_bm" topic="bm" robot_namespace="$(arg robot_namespace)"/>
+  <joint name="ultrasonic_mount_joint_bm" type="fixed">
+    <origin xyz="0.0 0.0 0.0" rpy="0 0 ${M_PI}"/>
+    <parent link="chassis_link"/>
+    <child link="base_ultrasonic_bm" />
+  </joint>
     <sick_lms1xx frame="base_laser" topic="scan" robot_namespace="$(arg robot_namespace)"/>
     <joint name="laser_mount_joint" type="fixed">

Commit message: Update README.md --- Add bin parking service --- Fix pi/4 offset in urdf

File: unicorn_description/urdf/unicorn_target_2.urdf.xacro (robot description, xacro)
@@ -18,5 +18,5 @@
   <!-- LMS111 -->
   <xacro:arg name="laser_xyz" default="0.0 0.0 0.5" />
-  <xacro:arg name="laser_rpy" default="0.0 0.0 ${M_PI}" />
+  <xacro:arg name="laser_rpy" default="0.0 0.0 ${M_PI-M_PI/4}" />
   <xacro:include filename="$(find lms1xx)/urdf/sick_lms1xx.urdf.xacro" />
   <!-- Ultrasonic sensor -->
@@ -274,10 +274,10 @@
   <origin xyz="0.27 0.0 0.0" rpy="0 0 0" />
   </joint> -->
-  <ultrasonic_sensor frame="base_ultrasonic_bm" topic="bm" robot_namespace="$(arg robot_namespace)"/>
+  <!-- <ultrasonic_sensor frame="base_ultrasonic_bm" topic="bm" robot_namespace="$(arg robot_namespace)"/>
   <joint name="ultrasonic_mount_joint_bm" type="fixed">
     <origin xyz="0.0 0.0 0.0" rpy="0 0 ${M_PI}"/>
     <parent link="chassis_link"/>
     <child link="base_ultrasonic_bm" />
-  </joint>
+  </joint> -->
     <sick_lms1xx frame="base_laser" topic="scan" robot_namespace="$(arg robot_namespace)"/>
     <joint name="laser_mount_joint" type="fixed">

Commit message: Add Range sensor layer

File: unicorn_description/urdf/unicorn_target_2.urdf.xacro (robot description, xacro)
@@ -227,57 +227,52 @@
   <swivel_wheel fb="front" lr="left" parent="chassis_link" translateY="-0.16" translateX="0.355" translateZ="0.03" wheel_radius="0.05" wheel_height="0.05" flip="0"/>
   <swivel_wheel fb="front" lr="right" parent="chassis_link" translateY="0.16" translateX="0.355" translateZ="0.03" wheel_radius="0.05" wheel_height="0.05" flip="0"/>
-  <!-- LOOP SENSORs -->
-  <!-- <sensorpos name="loop_front_center" parent="base_link" translateX="0.38" translateY="0.0" translateZ="-0.04"/>
-  <sensorpos name="loop_front_right" parent="base_link" translateX="0.38" translateY="-0.07" translateZ="-0.04"/>
-  <sensorpos name="loop_rear_left" parent="base_link" translateX="-0.07" translateY="0.14" translateZ="-0.04"/>
-  <sensorpos name="loop_rear_right" parent="base_link" translateX="-0.07" translateY="-0.14" translateZ="-0.04"/> -->
-  <!-- CONFINEMENT SENSORs -->
-  <!-- <sensorpos name="col_front_chassis" parent="base_link" translateX="0.55" translateY="0.0" translateZ="0.00"/>
-  <sensorpos name="col_front_left" parent="base_link" translateX="0.43" translateY="0.24" translateZ="0.00"/>
-  <sensorpos name="col_front_right" parent="base_link" translateX="0.43" translateY="-0.24" translateZ="0.00"/>
-  <sensorpos name="col_rear_left" parent="base_link" translateX="-0.10" translateY="0.24" translateZ="0.0"/>
-  <sensorpos name="col_rear_right" parent="base_link" translateX="-0.10" translateY="-0.24" translateZ="0.0"/> -->
-  <!-- CUTTING DISC -->
-  <!-- <link name="cutting_disc_center">
-    <visual>
-        <origin xyz="0 0 0" rpy="0 0 0" />
-        <geometry>
-            <cylinder length="0.01" radius="0.11" />
-        </geometry>
-        <material name="Purple" />
-    </visual>
-  </link>
-  <gazebo reference="cutting_disc_center">
-    <turnGravityOff>false</turnGravityOff>
-  </gazebo>
-  <joint name="cutting_disc_center_joint" type="fixed">
-    <parent link="base_link"/>
-    <child link="cutting_disc_center" />
-  <origin xyz="0.25 0.0 -0.07" rpy="0 0 0" />
-  </joint> -->
-  <!-- Antenna -->
-  <!-- <link name="antenna_center">
-    <visual>
-        <origin xyz="0 0 0" rpy="0 0 0" />
-        <geometry>
-            <cylinder length="0.01" radius="0.05" />
-        </geometry>
-        <material name="Purple" />
-    </visual>
-  </link>
-  <gazebo reference="antenna_center">
-    <turnGravityOff>false</turnGravityOff>
-  </gazebo>
-  <joint name="antenna_center_joint" type="fixed">
-    <parent link="base_link"/>
-    <child link="antenna_center" />
-  <origin xyz="0.27 0.0 0.0" rpy="0 0 0" />
-  </joint> -->
-  <!-- <ultrasonic_sensor frame="base_ultrasonic_bm" topic="bm" robot_namespace="$(arg robot_namespace)"/>
-  <joint name="ultrasonic_mount_joint_bm" type="fixed">
-    <origin xyz="0.0 0.0 0.0" rpy="0 0 ${M_PI}"/>
-    <parent link="chassis_link"/>
-    <child link="base_ultrasonic_bm" />
-  </joint> -->
+  <ultrasonic_sensor frame="base_ultrasonic_br" topic="br" robot_namespace="$(arg robot_namespace)"/>
+  <joint name="ultrasonic_mount_joint_br" type="fixed">
+    <origin xyz="0.4 0.25 0.0" rpy="0 0 ${M_PI/2}"/>
+    <parent link="chassis_link"/>
+    <child link="base_ultrasonic_br" />
+  </joint>
+  <ultrasonic_sensor frame="base_ultrasonic_bl" topic="bl" robot_namespace="$(arg robot_namespace)"/>
+  <joint name="ultrasonic_mount_joint_bl" type="fixed">
+    <origin xyz="0.4 -0.25 0.0" rpy="0 0 ${-M_PI/2}"/>
+    <parent link="chassis_link"/>
+    <child link="base_ultrasonic_bl" />
+  </joint>
+  <ultrasonic_sensor frame="base_ultrasonic_fl" topic="fl" robot_namespace="$(arg robot_namespace)"/>
+  <joint name="ultrasonic_mount_joint_fl" type="fixed">
+    <origin xyz="-0.2 -0.25 0.0" rpy="0 0 ${M_PI+M_PI/4}"/>
+    <parent link="chassis_link"/>
+    <child link="base_ultrasonic_fl" />
+  </joint>
+  <ultrasonic_sensor frame="base_ultrasonic_fr" topic="fr" robot_namespace="$(arg robot_namespace)"/>
+  <joint name="ultrasonic_mount_joint_fr" type="fixed">
+    <origin xyz="-0.2 0.25 0.0" rpy="0 0 ${M_PI-M_PI/4}"/>
+    <parent link="chassis_link"/>
+    <child link="base_ultrasonic_fr" />
+  </joint>
+  <ultrasonic_sensor frame="base_ultrasonic_bmr" topic="bmr" robot_namespace="$(arg robot_namespace)"/>
+  <joint name="ultrasonic_mount_joint_bmr" type="fixed">
+    <origin xyz="0.5 0.1 0.0" rpy="0 0 0"/>
+    <parent link="chassis_link"/>
+    <child link="base_ultrasonic_bmr" />
+  </joint>
+  <ultrasonic_sensor frame="base_ultrasonic_bml" topic="bml" robot_namespace="$(arg robot_namespace)"/>
+  <joint name="ultrasonic_mount_joint_bml" type="fixed">
+    <origin xyz="0.5 -0.1 0.0" rpy="0 0 0"/>
+    <parent link="chassis_link"/>
+    <child link="base_ultrasonic_bml" />
+  </joint>
+  <ultrasonic_sensor frame="base_ultrasonic_fmr" topic="fmr" robot_namespace="$(arg robot_namespace)"/>
+  <joint name="ultrasonic_mount_joint_fmr" type="fixed">
+    <origin xyz="-0.2 0.1 0.0" rpy="0 0 ${M_PI}"/>
+    <parent link="chassis_link"/>
+    <child link="base_ultrasonic_fmr" />
+  </joint>
+  <ultrasonic_sensor frame="base_ultrasonic_fml" topic="fml" robot_namespace="$(arg robot_namespace)"/>
+  <joint name="ultrasonic_mount_joint_fml" type="fixed">
+    <origin xyz="-0.2 -0.1 0.0" rpy="0 0 ${M_PI}"/>
+    <parent link="chassis_link"/>
+    <child link="base_ultrasonic_fml" />
+  </joint>
     <sick_lms1xx frame="base_laser" topic="scan" robot_namespace="$(arg robot_namespace)"/>
     <joint name="laser_mount_joint" type="fixed">

Commit message: Fix sonar layer on costmap

File: unicorn_description/urdf/unicorn_target_2.urdf.xacro (robot description, xacro)
@@ -229,5 +229,5 @@
   <ultrasonic_sensor frame="base_ultrasonic_br" topic="br" robot_namespace="$(arg robot_namespace)"/>
   <joint name="ultrasonic_mount_joint_br" type="fixed">
-    <origin xyz="0.4 0.25 0.0" rpy="0 0 ${M_PI/2}"/>
+    <origin xyz="0.45 0.2 0.0" rpy="0 0 ${3*M_PI/4}"/>
     <parent link="chassis_link"/>
     <child link="base_ultrasonic_br" />
@@ -235,5 +235,5 @@
   <ultrasonic_sensor frame="base_ultrasonic_bl" topic="bl" robot_namespace="$(arg robot_namespace)"/>
   <joint name="ultrasonic_mount_joint_bl" type="fixed">
-    <origin xyz="0.4 -0.25 0.0" rpy="0 0 ${-M_PI/2}"/>
+    <origin xyz="0.45 -0.2 0.0" rpy="0 0 ${-3*M_PI/4}"/>
     <parent link="chassis_link"/>
     <child link="base_ultrasonic_bl" />
@@ -241,5 +241,5 @@
   <ultrasonic_sensor frame="base_ultrasonic_fl" topic="fl" robot_namespace="$(arg robot_namespace)"/>
   <joint name="ultrasonic_mount_joint_fl" type="fixed">
-    <origin xyz="-0.2 -0.25 0.0" rpy="0 0 ${M_PI+M_PI/4}"/>
+    <origin xyz="-0.2 -0.25 0.0" rpy="0 0 ${5*M_PI/4}"/>
     <parent link="chassis_link"/>
     <child link="base_ultrasonic_fl" />
@@ -247,5 +247,5 @@
   <ultrasonic_sensor frame="base_ultrasonic_fr" topic="fr" robot_namespace="$(arg robot_namespace)"/>
   <joint name="ultrasonic_mount_joint_fr" type="fixed">
-    <origin xyz="-0.2 0.25 0.0" rpy="0 0 ${M_PI-M_PI/4}"/>
+    <origin xyz="-0.2 0.25 0.0" rpy="0 0 ${3*M_PI/4}"/>
     <parent link="chassis_link"/>
     <child link="base_ultrasonic_fr" />
@@ -253,5 +253,5 @@
   <ultrasonic_sensor frame="base_ultrasonic_bmr" topic="bmr" robot_namespace="$(arg robot_namespace)"/>
   <joint name="ultrasonic_mount_joint_bmr" type="fixed">
-    <origin xyz="0.5 0.1 0.0" rpy="0 0 0"/>
+    <origin xyz="0.47 0.15 0.0" rpy="0 0 ${-M_PI/6}"/>
     <parent link="chassis_link"/>
     <child link="base_ultrasonic_bmr" />
@@ -259,5 +259,5 @@
   <ultrasonic_sensor frame="base_ultrasonic_bml" topic="bml" robot_namespace="$(arg robot_namespace)"/>
   <joint name="ultrasonic_mount_joint_bml" type="fixed">
-    <origin xyz="0.5 -0.1 0.0" rpy="0 0 0"/>
+    <origin xyz="0.47 -0.15 0.0" rpy="0 0 ${M_PI/6}"/>
     <parent link="chassis_link"/>
     <child link="base_ultrasonic_bml" />

Commit message: Update ultrasonic driver, costmap params, local planner [tested & working]

File: unicorn_description/urdf/unicorn_target_2.urdf.xacro (robot description, xacro)
@@ -235,5 +235,5 @@
   <ultrasonic_sensor frame="base_ultrasonic_bl" topic="bl" robot_namespace="$(arg robot_namespace)"/>
   <joint name="ultrasonic_mount_joint_bl" type="fixed">
-    <origin xyz="0.45 -0.2 0.0" rpy="0 0 ${-3*M_PI/4}"/>
+    <origin xyz="0.45 -0.2 0.0" rpy="0 0 ${M_PI-55*M_PI/180}"/>
     <parent link="chassis_link"/>
     <child link="base_ultrasonic_bl" />
@@ -241,5 +241,5 @@
   <ultrasonic_sensor frame="base_ultrasonic_fl" topic="fl" robot_namespace="$(arg robot_namespace)"/>
   <joint name="ultrasonic_mount_joint_fl" type="fixed">
-    <origin xyz="-0.2 -0.25 0.0" rpy="0 0 ${5*M_PI/4}"/>
+    <origin xyz="-0.2 -0.25 0.0" rpy="0 0 ${M_PI+55*M_PI/180}"/>
     <parent link="chassis_link"/>
     <child link="base_ultrasonic_fl" />
