Commit message: Lower max vel x of teb local planner

File: unicorn_description/urdf/unicorn_target.urdf.xacro (robot description, xacro)
@@ -5,5 +5,5 @@
   <property name="M_PI" value="3.1415926535897931" />
   <xacro:arg name="laser_enabled" default="true" />
-  <xacro:arg name="laser_xyz" default="0.3206 0.0 0.310" />
+  <xacro:arg name="laser_xyz" default="0 0.0 0.310" />
   <xacro:arg name="laser_rpy" default="0.0 0.0 0.0" />
   <xacro:arg name="robot_namespace" default="/" />
@@ -33,5 +33,5 @@
     <inertial>
       <origin
-        xyz="0.17 0 -0.10"
+        xyz="0 0 -0.10"
         rpy="0 0 0" />
       <mass
@@ -41,5 +41,5 @@
     <visual>
       <origin
-        xyz="-0.17 0 0"
+        xyz="0 0 0"
         rpy="0 0 0" />
       <geometry>
@@ -55,5 +55,5 @@
     <collision>
       <origin
-        xyz="-0.17 0 0.08"
+        xyz="0 0 0.08"
         rpy="0 0 0" />
       <geometry>
@@ -95,5 +95,5 @@
         </visual>
     </link>
-    <link name="zed_right_camera">
+    <!-- <link name="zed_right_camera">
         <visual>
             <origin xyz="0 0 0" rpy="0 1.57 0"/>
@@ -105,5 +105,5 @@
             </material>
         </visual>
-    </link>
+    </link> -->
     <link name="zed_depth_camera" />
     <joint name="zed_left_camera_joint" type="fixed">
@@ -117,13 +117,13 @@
         <origin xyz="0 0 0" rpy="-1.5707963267948966 0 -1.5707963267948966" />
     </joint>
-    <joint name="zed_right_camera_joint" type="fixed">
+   <!--  <joint name="zed_right_camera_joint" type="fixed">
         <parent link="zed_center"/>
         <child link="zed_right_camera"/>
         <origin xyz="0 -0.06 0" rpy="0 0 0" />
-    </joint>
-    <joint name="zed_center_joint" type="fixed">
+    </joint> -->
+    <joint name="base_link_joint" type="fixed">
       <parent link="base_link"/>
       <child link="zed_center"/>
-      <origin xyz="0 0 0.3" rpy="${-M_PI/2} 0 0"/>
+      <origin xyz="0 0 0.3" rpy="0 0 0"/>
     </joint>
   <!-- WHEELs -->

Commit message: Cleanup + Commenting + Documenting + integrating am_driver_safe and zed-ros-wrapper. Added PID control to back into bin [working sim]

File: unicorn_description/urdf/unicorn_target.urdf.xacro (robot description, xacro)
@@ -1,26 +1,13 @@
 <?xml version="1.0"?>
-<robot name="automower" xmlns:xacro="http://www.ros.org/wiki/xacro">
+<robot name="unicorn" xmlns:xacro="http://www.ros.org/wiki/xacro">
   <!-- PROPERTY LIST -->
+  <xacro:arg name="robot_namespace" default="/" />
   <!--All units in m-kg-s-radians unit system -->
   <property name="M_PI" value="3.1415926535897931" />
-  <xacro:arg name="laser_enabled" default="true" />
-  <xacro:arg name="laser_xyz" default="0 0.0 0.310" />
-  <xacro:arg name="laser_rpy" default="0.0 0.0 0.0" />
-  <xacro:arg name="robot_namespace" default="/" />
-  <!-- Included URDF/XACRO Files -->
-  <xacro:include filename="$(find am_description)/urdf/materials.urdf.xacro" />
-  <xacro:include filename="$(find am_description)/urdf/wheel.urdf.xacro" />
-  <xacro:include filename="$(find am_description)/urdf/swivel_wheel.urdf.xacro" />
-  <xacro:include filename="$(find am_description)/urdf/sensorpos.urdf.xacro" />
-  <xacro:include filename="$(find lms1xx)/urdf/sick_lms1xx.urdf.xacro" />
-  <xacro:include filename="$(find unicorn_description)/urdf/stereo_camera.urdf.xacro" />
-  <!--<xacro:include filename="$(find husky_description)/urdf/accessories/sick_lms1xx_mount.urdf.xacro"/>-->
-  <!--<xacro:include filename="$(find husky_description)/urdf/accessories/sensor_arch.urdf.xacro"/>-->
   <!-- Main Body-base -->
   <property name="base_x_size" value="0.72" />
   <property name="base_y_size" value="0.55" />
-  <property name="base_z_size" value="0.23" />
-  <property name="base_mass" value="15" /> <!-- in kg-->
-  <property name="base_z_origin_to_wheel_origin" value="-0.07" />
+  <property name="base_z_size" value="0.6" />
+  <property name="base_mass" value="15" /> <!-- 21.446 in kg-->
   <!--Inertial macros for the box and cylinder. Units are kg*m^2-->
   <macro name="box_inertia" params="m x y z">
@@ -29,9 +16,23 @@
               izz="${m*(x*x+z*z)/12}" />
   </macro>
+  <!-- LMS111 -->
+  <xacro:arg name="laser_xyz" default="0.0 0.0 0.5" />
+  <xacro:arg name="laser_rpy" default="0.0 0.0 ${M_PI-M_PI/4}" />
+  <xacro:include filename="$(find lms1xx)/urdf/sick_lms1xx.urdf.xacro" />
+  <!-- Ultrasonic sensor -->
+  <xacro:arg name="ultrasonic_xyz" default="-0.3 0 0.2" />
+  <xacro:arg name="ultrasonic_rpy" default="0 0 0" />
+  <xacro:include filename="$(find unicorn_description)/urdf/ultrasonic_sensor.urdf.xacro" />
+  <!-- Wheel -->
+  <xacro:include filename="$(find am_description)/urdf/wheel.urdf.xacro" />
+  <!-- Swivel wheel -->
+  <xacro:include filename="$(find am_description)/urdf/swivel_wheel.urdf.xacro" />
+  <!-- Materials -->
+  <xacro:include filename="$(find am_description)/urdf/materials.urdf.xacro" />
   <link
     name="base_link">
     <inertial>
       <origin
-        xyz="0 0 0"
+        xyz="0.17 0 0"
         rpy="0 0 0" />
       <mass
@@ -41,5 +42,5 @@
     <visual>
       <origin
-        xyz="0 0 0"
+        xyz="-0.17 0 0"
         rpy="0 0 0" />
       <geometry>
@@ -55,5 +56,5 @@
     <collision>
       <origin
-        xyz="0 0 0.08"
+        xyz="-0.17 0 0.08"
         rpy="0 0 0" />
       <geometry>
@@ -69,8 +70,52 @@
     </collision>
   </link>
+  <link
+    name="chassis_link">
+    <inertial>
+      <origin
+        xyz="0 0 0"
+        rpy="0 0 0" />
+      <mass
+        value="0.01" />
+      <box_inertia  m="${5*0.01}" x="${base_x_size}" y="${base_y_size}" z="${base_z_size}"/>
+    </inertial>
+    <visual>
+      <origin
+        xyz="0 0 0"
+        rpy="0 0 0" />
+      <geometry>
+        <box size="0.01 0.01 0.01"/>
+      </geometry>
+      <material
+        name="">
+        <color
+          rgba="0.79216 0.81961 0.93333 1" />
+      </material>
+    </visual>
+    <collision>
+      <origin
+        xyz="0 0 0"
+        rpy="0 0 0" />
+      <geometry>
+        <!-- <mesh
+          filename="package://unicorn_description/meshes/base_link.STL" /> -->
+          <box size="0.01 0.01 0.01"/>
+      </geometry>
+      <!-- <surface>
+         <friction>
+           <ode><mu>0</mu><mu2>0</mu2></ode>
+         </friction>
+      </surface> -->
+    </collision>
+  </link>
   <gazebo reference="base_link_gazebo">
     <material>Gazebo/Green</material>
     <turnGravityOff>false</turnGravityOff>
   </gazebo>
+  <joint name="base_chassis_joint" type="fixed">
+    <parent link="base_link"/>
+    <child link="chassis_link" />
+  <origin xyz="0 0.0 0" rpy="0 0 ${M_PI}" />
+  </joint>
   <link name="zed_left_camera">
         <visual>
@@ -122,75 +167,118 @@
         <origin xyz="0 -0.06 0" rpy="0 0 0" />
     </joint> -->
-    <joint name="base_link_joint" type="fixed">
-      <parent link="base_link"/>
+    <joint name="chassis_zed_joint" type="fixed">
+      <parent link="chassis_link"/>
       <child link="zed_center"/>
-      <origin xyz="0 0 0.3" rpy="0 0 0"/>
+      <origin xyz="-0.2 0.0 0.3" rpy="0 0 ${-M_PI}"/>
     </joint>
-  <!-- WHEELs -->
-  <wheel fb="back" lr="right" parent="base_link" translateY="-0.24" translateX="0.0" translateZ="0.0" wheel_radius="0.1225" wheel_height="0.032" flip="1"/>
-  <wheel fb="back" lr="left" parent="base_link" translateY="0.24" translateX="0.0" translateZ="0.0" wheel_radius="0.1225" wheel_height="0.032" flip="1"/>
-<!--
-  <wheel fb="front" lr="right" parent="base_link" translateY="-0.15" translateX="0.35" translateZ="-0.065" wheel_radius="0.06" wheel_height="0.05" flip="1"/>
-  <wheel fb="front" lr="left" parent="base_link" translateY="0.15" translateX="0.35" translateZ="-0.065" wheel_radius="0.06" wheel_height="0.05" flip="1"/>
--->
-  <swivel_wheel fb="front" lr="right" parent="base_link" translateY="-0.16" translateX="0.355" translateZ="0.03" wheel_radius="0.05" wheel_height="0.05" flip="0"/>
-  <swivel_wheel fb="front" lr="left" parent="base_link" translateY="0.16" translateX="0.355" translateZ="0.03" wheel_radius="0.05" wheel_height="0.05" flip="0"/>
-  <!-- LOOP SENSORs -->
-  <sensorpos name="loop_front_center" parent="base_link" translateX="0.38" translateY="0.0" translateZ="-0.04"/>
-  <sensorpos name="loop_front_right" parent="base_link" translateX="0.38" translateY="-0.07" translateZ="-0.04"/>
-  <sensorpos name="loop_rear_left" parent="base_link" translateX="-0.07" translateY="0.14" translateZ="-0.04"/>
-  <sensorpos name="loop_rear_right" parent="base_link" translateX="-0.07" translateY="-0.14" translateZ="-0.04"/>
-  <!-- CONFINEMENT SENSORs -->
-  <sensorpos name="col_front_chassis" parent="base_link" translateX="0.55" translateY="0.0" translateZ="0.00"/>
-  <sensorpos name="col_front_left" parent="base_link" translateX="0.43" translateY="0.24" translateZ="0.00"/>
-  <sensorpos name="col_front_right" parent="base_link" translateX="0.43" translateY="-0.24" translateZ="0.00"/>
-  <sensorpos name="col_rear_left" parent="base_link" translateX="-0.10" translateY="0.24" translateZ="0.0"/>
-  <sensorpos name="col_rear_right" parent="base_link" translateX="-0.10" translateY="-0.24" translateZ="0.0"/>
-  <!-- CUTTING DISC -->
-  <link name="cutting_disc_center">
-    <visual>
-        <origin xyz="0 0 0" rpy="0 0 0" />
-        <geometry>
-            <cylinder length="0.01" radius="0.11" />
-        </geometry>
-        <material name="Purple" />
-    </visual>
+  <!-- Orbbec camera -->
+  <link name="camera_rgb_frame">
+      <visual>
+          <origin xyz="0 0 0" rpy="0 1.57 0"/>
+          <geometry>
+              <box size="0.01 0.01 0.01"/>
+          </geometry>
+          <material name="dark_grey">
+              <color rgba="0.1 0.1 0.1 1"/>
+          </material>
+      </visual>
   </link>
-  <gazebo reference="cutting_disc_center">
-    <turnGravityOff>false</turnGravityOff>
-  </gazebo>
-  <joint name="cutting_disc_center_joint" type="fixed">
-    <parent link="base_link"/>
-    <child link="cutting_disc_center" />
-	<origin xyz="0.25 0.0 -0.07" rpy="0 0 0" />
-  </joint>
-  <!-- Antenna -->
-  <link name="antenna_center">
-    <visual>
-        <origin xyz="0 0 0" rpy="0 0 0" />
-        <geometry>
-            <cylinder length="0.01" radius="0.05" />
-        </geometry>
-        <material name="Purple" />
-    </visual>
+  <link name="camera_link">
+      <visual>
+          <origin xyz="0 0 0" rpy="0 0 0"/>
+          <geometry>
+              <box size="0.01 0.01 0.01"/>
+          </geometry>
+          <material name="light_grey">
+              <color rgba="0.8 0.8 0.8 0.8"/>
+          </material>
+      </visual>
   </link>
-  <gazebo reference="antenna_center">
-    <turnGravityOff>false</turnGravityOff>
-  </gazebo>
-  <joint name="antenna_center_joint" type="fixed">
-    <parent link="base_link"/>
-    <child link="antenna_center" />
-	<origin xyz="0.27 0.0 0.0" rpy="0 0 0" />
-  </joint>
-  <!-- sick lms1xx -->
-  <xacro:if value="$(arg laser_enabled)">
-    <!--<sick_lms1xx_mount prefix="base"/>-->
+  <link name="camera_depth_frame" />
+  <link name="camera_depth_optical_frame" />
+  <link name="camera_rgb_optical_frame" />
+  <joint name="chassis_orbbec_joint" type="fixed">
+    <parent link="chassis_link"/>
+    <child link="camera_link"/>
+    <origin xyz="0.2 0 0.3" rpy="0 0 ${M_PI}"/>
+  </joint>
+  <joint name="orbbec_rgb_camera_joint" type="fixed">
+    <parent link="camera_link"/>
+    <child link="camera_rgb_frame"/>
+    <origin xyz="0 0.06 0" rpy="0 0 0" />
+  </joint>
+  <joint name="orbbec_depth_camera_joint" type="fixed">
+    <parent link="camera_link"/>
+    <child link="camera_depth_frame"/>
+    <origin xyz="0 0 0" rpy="-1.5707963267948966 0 -1.5707963267948966" />
+  </joint>
+  <joint name="orbbec_depth_optical_joint" type="fixed">
+    <parent link="camera_depth_frame"/>
+    <child link="camera_depth_optical_frame"/>
+    <origin xyz="0 0 0" rpy="0 0 0" />
+  </joint>
+  <joint name="orbbec_rgb_optical_joint" type="fixed">
+    <parent link="camera_rgb_frame"/>
+    <child link="camera_rgb_optical_frame"/>
+    <origin xyz="0 0 0" rpy="0 0 0" />
+  </joint>
+  <wheel fb="back" lr="left" parent="chassis_link" translateY="-0.24" translateX="0.0" translateZ="-0.006" wheel_radius="0.1225" wheel_height="0.032" flip="1"/>
+  <wheel fb="back" lr="right" parent="chassis_link" translateY="0.24" translateX="0.0" translateZ="-0.006" wheel_radius="0.1225" wheel_height="0.032" flip="1"/>
+  <swivel_wheel fb="front" lr="left" parent="chassis_link" translateY="-0.16" translateX="0.355" translateZ="0.03" wheel_radius="0.05" wheel_height="0.05" flip="0"/>
+  <swivel_wheel fb="front" lr="right" parent="chassis_link" translateY="0.16" translateX="0.355" translateZ="0.03" wheel_radius="0.05" wheel_height="0.05" flip="0"/>
+  <ultrasonic_sensor frame="base_ultrasonic_br" topic="br" robot_namespace="$(arg robot_namespace)"/>
+  <joint name="ultrasonic_mount_joint_br" type="fixed">
+    <origin xyz="0.45 0.2 0.0" rpy="0 0 ${3*M_PI/4}"/>
+    <parent link="chassis_link"/>
+    <child link="base_ultrasonic_br" />
+  </joint>
+  <ultrasonic_sensor frame="base_ultrasonic_bl" topic="bl" robot_namespace="$(arg robot_namespace)"/>
+  <joint name="ultrasonic_mount_joint_bl" type="fixed">
+    <origin xyz="0.45 -0.2 0.0" rpy="0 0 ${M_PI-55*M_PI/180}"/>
+    <parent link="chassis_link"/>
+    <child link="base_ultrasonic_bl" />
+  </joint>
+  <ultrasonic_sensor frame="base_ultrasonic_fl" topic="fl" robot_namespace="$(arg robot_namespace)"/>
+  <joint name="ultrasonic_mount_joint_fl" type="fixed">
+    <origin xyz="-0.2 -0.25 0.0" rpy="0 0 ${M_PI+55*M_PI/180}"/>
+    <parent link="chassis_link"/>
+    <child link="base_ultrasonic_fl" />
+  </joint>
+  <ultrasonic_sensor frame="base_ultrasonic_fr" topic="fr" robot_namespace="$(arg robot_namespace)"/>
+  <joint name="ultrasonic_mount_joint_fr" type="fixed">
+    <origin xyz="-0.2 0.25 0.0" rpy="0 0 ${3*M_PI/4}"/>
+    <parent link="chassis_link"/>
+    <child link="base_ultrasonic_fr" />
+  </joint>
+  <ultrasonic_sensor frame="base_ultrasonic_bmr" topic="bmr" robot_namespace="$(arg robot_namespace)"/>
+  <joint name="ultrasonic_mount_joint_bmr" type="fixed">
+    <origin xyz="0.47 0.15 0.0" rpy="0 0 ${-M_PI/6}"/>
+    <parent link="chassis_link"/>
+    <child link="base_ultrasonic_bmr" />
+  </joint>
+  <ultrasonic_sensor frame="base_ultrasonic_bml" topic="bml" robot_namespace="$(arg robot_namespace)"/>
+  <joint name="ultrasonic_mount_joint_bml" type="fixed">
+    <origin xyz="0.47 -0.15 0.0" rpy="0 0 ${M_PI/6}"/>
+    <parent link="chassis_link"/>
+    <child link="base_ultrasonic_bml" />
+  </joint>
+  <ultrasonic_sensor frame="base_ultrasonic_fmr" topic="fmr" robot_namespace="$(arg robot_namespace)"/>
+  <joint name="ultrasonic_mount_joint_fmr" type="fixed">
+    <origin xyz="-0.2 0.1 0.0" rpy="0 0 ${M_PI}"/>
+    <parent link="chassis_link"/>
+    <child link="base_ultrasonic_fmr" />
+  </joint>
+  <ultrasonic_sensor frame="base_ultrasonic_fml" topic="fml" robot_namespace="$(arg robot_namespace)"/>
+  <joint name="ultrasonic_mount_joint_fml" type="fixed">
+    <origin xyz="-0.2 -0.1 0.0" rpy="0 0 ${M_PI}"/>
+    <parent link="chassis_link"/>
+    <child link="base_ultrasonic_fml" />
+  </joint>
     <sick_lms1xx frame="base_laser" topic="scan" robot_namespace="$(arg robot_namespace)"/>
     <joint name="laser_mount_joint" type="fixed">
       <origin xyz="$(arg laser_xyz)" rpy="$(arg laser_rpy)" />
-      <parent link="base_link" />
+      <parent link="chassis_link" />
       <child link="base_laser" />
     </joint>
-  </xacro:if>
   <!-- GAZEBO STUFF -->
   <gazebo>
@@ -206,5 +294,5 @@
       <odometryTopic>odom</odometryTopic>
       <odometryFrame>odom_gazebo</odometryFrame>
-      <robotBaseFrame>base_link_gazebo</robotBaseFrame>
+      <robotBaseFrame>chassis_link_gazebo</robotBaseFrame>
       <publishWheelTF>false</publishWheelTF>
       <publishWheelJointState>false</publishWheelJointState>
@@ -212,6 +300,6 @@
     <plugin name="gazebo_ros_control" filename="libgazebo_ros_control.so" />
     <plugin name="imu_plugin" filename="libhector_gazebo_ros_imu.so">
-    <alwaysOn>true</alwaysOn>
-    <bodyName>base_link</bodyName>
+    <alwaysOn>false</alwaysOn>
+    <bodyName>chassis_link_gazebo</bodyName>
     <topicName>imu</topicName>
     <serviceName>imu_service</serviceName>
@@ -219,50 +307,22 @@
     <rpyOffsets>0 0 0</rpyOffsets> <!-- deprecated -->
 <!--
-	    <gaussianNoise>0.0</gaussianNoise>
-	    <accelDrift>0.5 0.5 0.5</accelDrift>
-	    <accelGaussianNoise>0.35 0.35 0.3</accelGaussianNoise>
-	    <rateDrift>0.1 0.1 0.1</rateDrift>
-	    <rateGaussianNoise>0.05 0.05 0.015</rateGaussianNoise>
-	    <headingDrift>0.1</headingDrift>
-	    <headingGaussianNoise>1.00</headingGaussianNoise>
+      <gaussianNoise>0.0</gaussianNoise>
+      <accelDrift>0.5 0.5 0.5</accelDrift>
+      <accelGaussianNoise>0.35 0.35 0.3</accelGaussianNoise>
+      <rateDrift>0.1 0.1 0.1</rateDrift>
+      <rateGaussianNoise>0.05 0.05 0.015</rateGaussianNoise>
+      <headingDrift>0.1</headingDrift>
+      <headingGaussianNoise>1.00</headingGaussianNoise>
 -->
-		<gaussianNoise>0.0</gaussianNoise>  <!-- deprecated -->
-	    <accelDrift>0.0 0.0 0.0</accelDrift>
-	    <accelGaussianNoise>0.0 0.0 0.0</accelGaussianNoise>
-	    <rateDrift>0.0 0.0 0.0</rateDrift>
-	    <rateGaussianNoise>0.0 0.0 0.0</rateGaussianNoise>
-	    <headingDrift>0.0</headingDrift>
-	    <headingGaussianNoise>0.00</headingGaussianNoise>
+    <gaussianNoise>0.0</gaussianNoise>  <!-- deprecated -->
+      <accelDrift>0.0 0.0 0.0</accelDrift>
+      <accelGaussianNoise>0.0 0.0 0.0</accelGaussianNoise>
+      <rateDrift>0.0 0.0 0.0</rateDrift>
+      <rateGaussianNoise>0.0 0.0 0.0</rateGaussianNoise>
+      <headingDrift>0.0</headingDrift>
+      <headingGaussianNoise>0.00</headingGaussianNoise>
     </plugin>
     <plugin name="am_gazebo_wheelencoder" filename="libam_gazebo_wheelencoder.so">
-	</plugin>
-    <plugin name="automower_gps_sim" filename="libhector_gazebo_ros_gps.so">
-	  <alwaysOn>true</alwaysOn>
-	  <updateRate>4.0</updateRate>
-	  <bodyName>base_link</bodyName>
-	  <topicName>fix</topicName>
-	  <velocityTopicName>fix_vel</velocityTopicName>
-	  <drift>5.0 5.0 5.0</drift>
-	  <gaussianNoise>0.1 0.1 0.1</gaussianNoise>
-	  <velocityDrift>0 0 0</velocityDrift>
-	  <velocityGaussianNoise>0.1 0.1 0.1</velocityGaussianNoise>
-    </plugin>
-  </gazebo>
-  <gazebo reference="base_link">
-	<sensor name="automower_sensor" type="contact">
-		<always_on>true</always_on>
-		<update_rate>50</update_rate>
-		<contact>
-			<collision>base_link_collision</collision>
-		</contact>
-		<plugin name="automower_sensors_plugin" filename="libam_gazebo_sensors.so">
-			<always_on>true</always_on>
-			<update_rate>20</update_rate>
-			<bumperTopicName>sensor_status</bumperTopicName>
-			<loopTopicName>loop</loopTopicName>
-			<!-- 0x01 = FC, 0x02 = FR, 0x04 = RL, 0x08 = RR -->
-			<loopOutsideSensors>15</loopOutsideSensors>
-		</plugin>
-	</sensor>
+  </plugin>
   </gazebo>
 </robot>
